File: examples/triac-out/triac-out.kicad_sch (KiCad schematic)
At the start: 13 parts, among them Q1 Triac, U1 MOC3021M

Commit message: Added examples.
Parts:
- added J1: Power, TerminalBlock_Phoenix:TerminalBlock_Phoenix_MKDS-1,5-3-5.08_1x03_P5.08mm_Horizontal, symbol Connector_Generic:Conn_01x03
- added J2: DC_in, TerminalBlock_Phoenix:TerminalBlock_Phoenix_MKDS-1,5-2-5.08_1x02_P5.08mm_Horizontal, symbol Connector_Generic:Conn_01x02
- C1: footprint (none) -> Capacitor_THT:C_Axial_L3.8mm_D2.6mm_P10.00mm_Horizontal
- C2: footprint Capacitor_THT:CP_Axial_L10.0mm_D4.5mm_P15.00mm_Horizontal -> Capacitor_THT:C_Axial_L3.8mm_D2.6mm_P10.00mm_Horizontal
- RLoad1, V1, V2: now left out of the parts list
Connections:
- net GND: now also J1.3 (Pin_3); no longer D1.1 (K), U1.2, V1.2
- net Load: now also J1.2 (Pin_2)
- net Vin: now also J2.1 (Pin_1)
- net Net renamed Phase
- net Phase: now also J1.1 (Pin_1)
- new net GND1: D1.1 (K), J2.2 (Pin_2), U1.2, V1.2
Other:
- note added: ".tran 1m 20ms"
- note removed: ".tran 1u 20ms"
